Commit message: added colors

File: linorobot2_description/urdf/mech/base.urdf.xacro (robot description, xacro)
@@ -10,6 +10,6 @@
           <!-- <mesh filename="" scale="0.001 0.001 0.001"/> -->
         </geometry>
-        <material name="white">
-          <color rgba="1.0 1.0 1.0 1.0"/>
+        <material name="yellow">
+          <color rgba="0.8784 0.6627 0.6627 1.0"/>
         </material>
       </visual>
@@ -28,4 +28,14 @@
       </inertial>
     </link>
+    <gazebo reference="base_link">
+      <visual>
+        <material>
+          <ambient>0.8392 0.6314 0.0 1.0</ambient>
+          <diffuse>0.8392 0.6314 0.0 1.0</diffuse>
+          <specular>0.99 0.99 0.99 1.0</specular>
+          <emissive>0.0 0.0 0.0 0.0</emissive>
+        </material>
+      </visual>  rgb(214,161,0)
+    </gazebo>
     <joint name="base_to_footprint" type="fixed">
       <parent link="base_footprint"/>

File: linorobot2_description/urdf/mech/wheel.urdf.xacro (robot description, xacro)
@@ -8,6 +8,6 @@
           <cylinder radius="${radius}" length="${width}"/>
         </geometry>
-        <material name="black">
-            <color rgba="0.0 0.0 0.0 1.0"/>
+        <material name="blue">
+            <color rgba="0.1764 0.4588 0.8509 1.0"/>
         </material>
       </visual>
@@ -26,4 +26,14 @@
         </inertial>
     </link>
+    <gazebo reference="${side}_wheel_link">
+      <visual>
+        <material>
+          <ambient>0.1764 0.4588 0.8509 1.0</ambient>
+          <diffuse>0.1764 0.4588 0.8509 1.0</diffuse>
+          <specular>0.1764 0.4588 0.8509 1.0</specular>
+          <emissive>0.0 0.0 0.0 0.0</emissive>
+        </material>
+      </visual>
+    </gazebo>
     <joint name="${side}_wheel_joint" type="continuous">
       <axis xyz="0 1 0" />

Commit message: cleaned up

File: linorobot2_description/urdf/mech/base.urdf.xacro (robot description, xacro)
@@ -36,5 +36,5 @@
           <emissive>0.0 0.0 0.0 0.0</emissive>
         </material>
-      </visual>  rgb(214,161,0)
+      </visual>
     </gazebo>
     <joint name="base_to_footprint" type="fixed">
