Commit message: added spacing for readability

File: linorobot2_description/urdf/mech/caster_wheel.urdf.xacro (robot description, xacro)
@@ -31,5 +31,5 @@
                  iyy="${(2/5) * mass * (caster_wheel_radius * caster_wheel_radius)}" iyz="0"
                  izz="${(2/5) * mass * (caster_wheel_radius * caster_wheel_radius)}" />
-        </inertial>
+      </inertial>
     </link>
     <joint name="${side}_caster_wheel_joint" type="fixed">

File: linorobot2_description/urdf/mech/wheel.urdf.xacro (robot description, xacro)
@@ -24,5 +24,5 @@
                  iyy="${(2/5) * mass * (radius * radius)}" iyz="0"
                  izz="${(2/5) * mass * (radius * radius)}" />
-        </inertial>
+      </inertial>
     </link>
     <gazebo reference="${side}_wheel_link">
