Commit message: revert the geometry from sphere to cylinder

File: linorobot2_description/urdf/mech/mecanum_wheel.urdf.xacro (robot description, xacro)
@@ -1,4 +1,4 @@
 <?xml version="1.0"?>
-<robot xmlns:xacro="http://ros.org/wiki/xacro">
+<robot xmlns:xacro="http://ros.org/wiki/xacro" xmlns:gz="http://gazebosim.org/schema">
   <xacro:macro name="mecanum_wheel" params="side radius width pos_x pos_y pos_z mass mesh_file">
     <link name="${side}_wheel_link">
@@ -20,6 +20,5 @@
         <origin xyz="0 0 0" rpy="${pi/2} 0 0"/>
         <geometry>
-          <sphere radius="${radius}"/>
-          <!-- <cylinder radius="${radius}" length="${width}"/> -->
+          <cylinder radius="${radius}" length="${width}"/>
         </geometry>
       </collision>
@@ -33,6 +32,28 @@
     </link>
     <gazebo reference="${side}_wheel_link">
-        <mu1>0.01</mu1>
-        <mu2>0.01</mu2>
+      <collision>
+        <surface>
+          <friction>
+            <ode>
+              <mu>1.5</mu>
+              <mu2>0.7</mu2>
+              <kp>200000.0</kp>
+              <kd>5000.0</kd>
+              <xacro:if value="${side == 'front_left'}">
+                <fdir1 gz:expressed_in="base_footprint">1 -1 0</fdir1>
+              </xacro:if>
+              <xacro:if value="${side == 'rear_left'}">
+                <fdir1 gz:expressed_in="base_footprint">1 1 0</fdir1>
+              </xacro:if>
+              <xacro:if value="${side == 'front_right'}">
+                <fdir1 gz:expressed_in="base_footprint">1 1 0</fdir1>
+              </xacro:if>
+              <xacro:if value="${side == 'rear_right'}">
+                <fdir1 gz:expressed_in="base_footprint">1 -1 0</fdir1>
+              </xacro:if>
+            </ode>
+          </friction>
+        </surface>
+      </collision>
     </gazebo>
     <gazebo reference="${side}_wheel_link">
