Commit message: added visual

File: linorobot2_description/urdf/sensors/laser.urdf.xacro (robot description, xacro)
@@ -2,5 +2,38 @@
   <xacro:property name="M_PI" value="3.1415926535897931" />
   <xacro:macro name="laser" params="*origin update_rate ray_count min_angle max_angle min_range max_range">
-    <link name="laser"/>
+    <link name="laser">
+      <visual>
+        <origin xyz="0 0 -0.025" rpy="0 0 0"/>
+        <geometry>
+          <cylinder radius="0.0375" length="0.05"/>
+        </geometry>
+        <material name="green">
+            <color rgba="0.003 0.639 0.223 1.0"/>
+        </material>
+      </visual>
+      <collision>
+        <origin xyz="0 0 0" rpy="${pi/2} 0 0"/>
+        <geometry>
+          <cylinder radius="0.0375" length="0.05"/>
+        </geometry>
+      </collision>
+      <inertial>
+        <origin xyz="0 0 0" rpy="0 0 0"/>
+        <mass value="0.1"/>
+        <inertia ixx="${(2/5) * 0.1 * (0.0375 * 0.0375)}" ixy="0" ixz="0"
+                 iyy="${(2/5) * 0.1 * (0.0375 * 0.0375)}" iyz="0"
+                 izz="${(2/5) * 0.1 * (0.0375 * 0.0375)}" />
+      </inertial>
+    </link>
+    <gazebo reference="laser">
+      <visual>
+        <material>
+          <ambient>0.003 0.639 0.223 1.0</ambient>
+          <diffuse>0.003 0.639 0.223 1.0</diffuse>
+          <specular>0.003 0.639 0.223 1.0</specular>
+          <emissive>0.0 0.0 0.0 0.0</emissive>
+        </material>
+      </visual>
+    </gazebo>
     <joint name="laser_to_base_link" type="fixed">
       <parent link="base_link"/>

Commit message: exposed frame_id and topic_name

File: linorobot2_description/urdf/sensors/laser.urdf.xacro (robot description, xacro)
@@ -1,6 +1,6 @@
 <robot xmlns:xacro="http://ros.org/wiki/xacro">
   <xacro:property name="M_PI" value="3.1415926535897931" />
-  <xacro:macro name="laser" params="*origin update_rate ray_count min_angle max_angle min_range max_range">
-    <link name="laser">
+  <xacro:macro name="laser" params="*origin update_rate ray_count min_angle max_angle min_range max_range frame_id topic_name">
+    <link name="${frame_id}">
       <visual>
         <origin xyz="0 0 -0.025" rpy="0 0 0"/>
@@ -26,5 +26,5 @@
       </inertial>
     </link>
-    <gazebo reference="laser">
+    <gazebo reference="${frame_id}">
       <visual>
         <material>
@@ -36,10 +36,10 @@
       </visual>
     </gazebo>
-    <joint name="laser_to_base_link" type="fixed">
+    <joint name="${frame_id}_to_base_link" type="fixed">
       <parent link="base_link"/>
-      <child link="laser"/>
+      <child link="${frame_id}"/>
       <xacro:insert_block name="origin" />
     </joint>
-    <gazebo reference="laser">
+    <gazebo reference="${frame_id}">
       <sensor type="ray" name="head_hokuyo_sensor">
         <always_on>true</always_on>
@@ -64,11 +64,11 @@
         <plugin name="gazebo_ros_head_hokuyo_controller" filename="libgazebo_ros_ray_sensor.so">
           <ros>
-            <argument>~/out:=scan</argument>
+            <argument>~/out:=${topic_name}</argument>
           </ros>
           <output_type>sensor_msgs/LaserScan</output_type>
           <alwaysOn>true</alwaysOn>
           <updateRate>${update_rate}</updateRate>
-          <topicName>scan</topicName>
-          <frame_name>laser</frame_name>
+          <topicName>${topic_name}</topicName>
+          <frame_name>${frame_id}</frame_name>
           <output_type>sensor_msgs/LaserScan</output_type>
         </plugin>
