Commit message: simulate camera in gazebo

File: linorobot2_description/urdf/sensors/camera.urdf.xacro (robot description, xacro)
@@ -51,9 +51,12 @@
     <!-- https://github.com/ros-simulation/gazebo_ros_pkgs/wiki/ROS-2-Migration:-Camera#gazebo_ros_camera -->
     <gazebo reference="camera_link">
-      <sensor name="camera" type="depth">
-        <always_on>true</always_on>
-        <update_rate>30.0</update_rate>
+      <material>Gazebo/Black</material>
+      <sensor name="camera" type="camera">
+        <pose>  0 0 0 0 0 0</pose>
+        <update_rate>24.0</update_rate>
+        <visualize>true</visualize>
         <camera name="camera">
-          <horizontal_fov>1.50098</horizontal_fov>
+          <!-- TODO find info about webcam -->
+          <horizontal_fov>1.0</horizontal_fov>
           <image>
             <width>640</width>
@@ -61,21 +64,11 @@
             <format>R8G8B8</format>
           </image>
+          <clip>
+            <near>0.05</near>
+            <far>8</far>
+          </clip>
         </camera>
         <plugin name="camera_controller" filename="libgazebo_ros_camera.so">
-          <ros>
-            <remapping>/camera/camera_info:=/camera/color/camera_info</remapping>
-            <remapping>/camera/image_raw:=/camera/color/image_raw</remapping>
-            <remapping>/camera/points:=/camera/depth/color/points</remapping>
-            <remapping>/camera/depth/image_raw:=/camera/depth/image_rect_raw</remapping>
-          </ros>
-          <min_depth>0.015</min_depth>
-          <max_depth>3.0</max_depth>
-          <hack_baseline>0.07</hack_baseline>
-          <frame_name>camera_depth_link</frame_name>
-          <distortion_k1>0.00000001</distortion_k1>
-          <distortion_k2>0.00000001</distortion_k2>
-          <distortion_k3>0.00000001</distortion_k3>
-          <distortion_t1>0.00000001</distortion_t1>
-          <distortion_t2>0.00000001</distortion_t2>
+          <frame_name>camera_link_optical</frame_name>
         </plugin>
       </sensor>
