Commit message: renamed base laser

File: linorobot2_description/urdf/robots/square.urdf.xacro (robot description, xacro)
@@ -78,7 +78,7 @@
     <xacro:insert_block name="laser_pose" />
   </xacro:generic_laser>
-  <xacro:generic_laser_base>
+  <xacro:generic_base_laser>
     <xacro:insert_block name="base_laser_pose" />
-  </xacro:generic_laser_base>
+  </xacro:generic_base_laser>
   <xacro:depth_sensor>
     <xacro:insert_block name="depth_sensor_pose" />

File: linorobot2_description/urdf/sensors/generic_laser.urdf.xacro (robot description, xacro)
@@ -16,5 +16,5 @@
     </xacro:laser>
   </xacro:macro>
-  <xacro:macro name="generic_laser_base" params="*origin">
+  <xacro:macro name="generic_base_laser" params="*origin">
     <xacro:include filename="$(find linorobot2_description)/urdf/sensors/laser.urdf.xacro" />
     <xacro:laser

Commit message: fixed com problem

File: linorobot2_description/urdf/robots/square.urdf.xacro (robot description, xacro)
@@ -12,5 +12,5 @@
   <xacro:property name="wheel_mass" value=".1" />
   <xacro:property name="wheel_torque" value="20" />
-  <xacro:property name="front_caster_wheel" value="true" />
+  <xacro:property name="front_caster_wheel" value="false" />
   <xacro:property name="rear_caster_wheel" value="true" />
   <xacro:include filename="$(find linorobot2_description)/urdf/mech/base.urdf.xacro" />
@@ -25,5 +25,5 @@
   </xacro:property>
   <xacro:property name="base_laser_pose">
-    <origin xyz="0.08 0 -0.055" rpy="-3.1416 0 0"/>
+    <origin xyz="0.08 0 -0.05" rpy="-3.1416 0 0"/>
   </xacro:property>
   <xacro:property name="depth_sensor_pose">
