Commit message: update laser pose

File: linorobot2_description/urdf/4wd_properties.urdf.xacro (robot description, xacro)
@@ -13,5 +13,5 @@
   <xacro:property name="wheel_torque" value="20" />
   <xacro:property name="laser_pose">
-    <origin xyz="0 0 0.5" rpy="0 0 0"/>
+    <origin xyz="-0.0475 0 0.125" rpy="0 0 0"/>
   </xacro:property>
 </robot>

Commit message: updated sensor pose

File: linorobot2_description/urdf/4wd_properties.urdf.xacro (robot description, xacro)
@@ -16,5 +16,5 @@
   </xacro:property>
   <xacro:property name="depth_sensor_pose">
-    <origin xyz="0.2375 0 0.06" rpy="0 0 0"/>
+    <origin xyz="-0.065 0 0.255" rpy="0 0 0"/>
   </xacro:property>
 </robot>

Commit message: match catbot physical params

File: linorobot2_description/urdf/4wd_properties.urdf.xacro (robot description, xacro)
@@ -1,17 +1,17 @@
 <?xml version="1.0"?>
 <robot xmlns:xacro="http://ros.org/wiki/xacro">
-  <xacro:property name="base_length" value="0.445" />
-  <xacro:property name="base_width" value="0.200" />
-  <xacro:property name="base_height" value="0.129" />
-  <xacro:property name="base_mass" value="10" />
-  <xacro:property name="wheel_radius" value="0.07162" />
-  <xacro:property name="wheel_width" value="0.05" />
-  <xacro:property name="wheel_pos_x" value="0.120" />
-  <xacro:property name="wheel_pos_y" value="0.1355" />
-  <xacro:property name="wheel_pos_z" value="-0.04788" />
-  <xacro:property name="wheel_mass" value=".6" />
+  <xacro:property name="base_length" value="0.242" />
+  <xacro:property name="base_width" value="0.126" />
+  <xacro:property name="base_height" value="0.064" />
+  <xacro:property name="base_mass" value="2.05196" />
+  <xacro:property name="wheel_radius" value="0.033" />
+  <xacro:property name="wheel_width" value="0.0265" />
+  <xacro:property name="wheel_pos_x" value="0.087" />
+  <xacro:property name="wheel_pos_y" value="0.08" />
+  <xacro:property name="wheel_pos_z" value="-0.06" />
+  <xacro:property name="wheel_mass" value=".054378" />
   <xacro:property name="wheel_torque" value="20" />
   <xacro:property name="laser_pose">
-    <origin xyz="-0.0475 0 0.125" rpy="0 0 0"/>
+    <origin xyz="0.08 0 0.122" rpy="0 0 0"/>
   </xacro:property>
   <xacro:property name="depth_sensor_pose">

Commit message: removed depth camera and added urdf position of webcam

File: linorobot2_description/urdf/4wd_properties.urdf.xacro (robot description, xacro)
@@ -15,6 +15,9 @@
     <origin xyz="0.08 0 0.122" rpy="0 0 0"/>
   </xacro:property>
-  <xacro:property name="depth_sensor_pose">
+  <!-- <xacro:property name="depth_sensor_pose">
     <origin xyz="-0.065 0 0.255" rpy="0 0 0"/>
+  </xacro:property> -->
+  <xacro:property name="camera_pose">
+    <origin xyz="0.134 0 0.02" rpy="0 0 0"/>
   </xacro:property>
 </robot>
