Commit message: expose lidar pose in properties xacro

File: linorobot2_description/urdf/2wd_properties.urdf.xacro (robot description, xacro)
@@ -12,3 +12,6 @@
   <xacro:property name="wheel_mass" value=".1" />
   <xacro:property name="wheel_torque" value="20" />
+  <xacro:property name="laser_pose">
+    <origin xyz="0 0 0.1" rpy="0 0 0"/>
+  </xacro:property>
 </robot>

File: linorobot2_description/urdf/4wd_properties.urdf.xacro (robot description, xacro)
@@ -12,3 +12,6 @@
   <xacro:property name="wheel_mass" value=".6" />
   <xacro:property name="wheel_torque" value="20" />
+  <xacro:property name="laser_pose">
+    <origin xyz="0 0 0.5" rpy="0 0 0"/>
+  </xacro:property>
 </robot>

File: linorobot2_description/urdf/robots/2wd.urdf.xacro (robot description, xacro)
@@ -50,5 +50,5 @@
   <xacro:imu/>
   <xacro:ld06>
-    <origin xyz="0 0 0.1" rpy="0 0 0"/>
+    <xacro:insert_block name="laser_pose" />
   </xacro:ld06>
   <xacro:diff_drive_controller

File: linorobot2_description/urdf/robots/4wd.urdf.xacro (robot description, xacro)
@@ -53,5 +53,5 @@
   <xacro:imu/>
   <xacro:ld06>
-    <origin xyz="0 0 0.2" rpy="0 0 0"/>
+    <xacro:insert_block name="laser_pose" />
   </xacro:ld06>
   <xacro:diff_drive_controller

Commit message: expose adding of caster wheels on 2wd property

File: linorobot2_description/urdf/2wd_properties.urdf.xacro (robot description, xacro)
@@ -7,9 +7,11 @@
   <xacro:property name="wheel_radius" value="0.045" />
   <xacro:property name="wheel_width" value="0.01" />
-  <xacro:property name="wheel_pos_x" value="0.0415" />
+  <xacro:property name="wheel_pos_x" value="-0.0415" />
   <xacro:property name="wheel_pos_y" value="0.1" />
   <xacro:property name="wheel_pos_z" value="0.023" />
   <xacro:property name="wheel_mass" value=".1" />
   <xacro:property name="wheel_torque" value="20" />
+  <xacro:property name="front_caster_wheel" value="true" />
+  <xacro:property name="rear_caster_wheel" value="true" />
   <xacro:property name="laser_pose">
     <origin xyz="0 0 0.1" rpy="0 0 0"/>

File: linorobot2_description/urdf/robots/2wd.urdf.xacro (robot description, xacro)
@@ -34,18 +34,22 @@
     mass="${wheel_mass}"
   />
-  <!-- <xacro:caster_wheel
-    side="front"
-    mass="0.1"
-    base_length="${base_length}"
-    wheel_radius="${wheel_radius}"
-    wheel_pos_z="${wheel_pos_z}"
-  /> -->
-  <xacro:caster_wheel
-    side="rear"
-    mass="0.1"
-    base_length="${base_length}"
-    wheel_radius="${wheel_radius}"
-    wheel_pos_z="${wheel_pos_z}"
-  />
+  <xacro:if value="${front_caster_wheel}">
+    <xacro:caster_wheel
+      side="front"
+      mass="0.1"
+      base_length="${base_length}"
+      wheel_radius="${wheel_radius}"
+      wheel_pos_z="${wheel_pos_z}"
+    />
+  </xacro:if>
+  <xacro:if value="${rear_caster_wheel}">
+    <xacro:caster_wheel
+      side="rear"
+      mass="0.1"
+      base_length="${base_length}"
+      wheel_radius="${wheel_radius}"
+      wheel_pos_z="${wheel_pos_z}"
+    />
+  </xacro:if>
   <xacro:imu/>
   <xacro:ld06>

Commit message: added depth sensor placeholder

File: linorobot2_description/urdf/2wd_properties.urdf.xacro (robot description, xacro)
@@ -13,7 +13,10 @@
   <xacro:property name="wheel_torque" value="20" />
   <xacro:property name="front_caster_wheel" value="true" />
-  <xacro:property name="rear_caster_wheel" value="true" />
+  <xacro:property name="rear_caster_wheel" value="false" />
   <xacro:property name="laser_pose">
     <origin xyz="0 0 0.1" rpy="0 0 0"/>
   </xacro:property>
+  <xacro:property name="depth_sensor_pose">
+    <origin xyz="0.085 0 0.02" rpy="0 0 0"/>
+  </xacro:property>
 </robot>

File: linorobot2_description/urdf/4wd_properties.urdf.xacro (robot description, xacro)
@@ -15,3 +15,6 @@
     <origin xyz="-0.0475 0 0.125" rpy="0 0 0"/>
   </xacro:property>
+  <xacro:property name="depth_sensor_pose">
+    <origin xyz="0.2375 0 0.06" rpy="0 0 0"/>
+  </xacro:property>
 </robot>

File: linorobot2_description/urdf/robots/2wd.urdf.xacro (robot description, xacro)
@@ -7,4 +7,5 @@
   <xacro:include filename="$(find linorobot2_description)/urdf/sensors/imu.urdf.xacro" />
   <xacro:include filename="$(find linorobot2_description)/urdf/sensors/ld06.urdf.xacro" />
+  <xacro:include filename="$(find linorobot2_description)/urdf/sensors/depth_sensor.urdf.xacro" />
   <xacro:include filename="$(find linorobot2_description)/urdf/controllers/diff_drive.urdf.xacro" />
   <xacro:base
@@ -56,4 +57,7 @@
     <xacro:insert_block name="laser_pose" />
   </xacro:ld06>
+  <xacro:depth_sensor>
+    <xacro:insert_block name="depth_sensor_pose" />
+  </xacro:depth_sensor>
   <xacro:diff_drive_controller
     wheel_separation="${wheel_pos_y * 2}"

File: linorobot2_description/urdf/robots/4wd.urdf.xacro (robot description, xacro)
@@ -6,4 +6,5 @@
   <xacro:include filename="$(find linorobot2_description)/urdf/sensors/imu.urdf.xacro" />
   <xacro:include filename="$(find linorobot2_description)/urdf/sensors/ld06.urdf.xacro" />
+  <xacro:include filename="$(find linorobot2_description)/urdf/sensors/depth_sensor.urdf.xacro" />
   <xacro:include filename="$(find linorobot2_description)/urdf/controllers/skid_steer.urdf.xacro" />
   <xacro:base
@@ -55,4 +56,7 @@
     <xacro:insert_block name="laser_pose" />
   </xacro:ld06>
+  <xacro:depth_sensor>
+    <xacro:insert_block name="depth_sensor_pose" />
+  </xacro:depth_sensor>
   <xacro:diff_drive_controller
     wheel_separation="${wheel_pos_y * 2}"

File: linorobot2_description/urdf/robots/mecanum.urdf.xacro (robot description, xacro)
@@ -1,9 +1,10 @@
 <?xml version="1.0"?>
 <robot name="linorobot2_2wd" xmlns:xacro="http://ros.org/wiki/xacro">
-  <xacro:include filename="$(find linorobot2_description)/urdf/4wd_properties.urdf.xacro" />
+  <xacro:include filename="$(find linorobot2_description)/urdf/mecanum_properties.urdf.xacro" />
   <xacro:include filename="$(find linorobot2_description)/urdf/mech/base.urdf.xacro" />
   <xacro:include filename="$(find linorobot2_description)/urdf/mech/wheel.urdf.xacro" />
   <xacro:include filename="$(find linorobot2_description)/urdf/sensors/imu.urdf.xacro" />
   <xacro:include filename="$(find linorobot2_description)/urdf/sensors/ld06.urdf.xacro" />
+  <xacro:include filename="$(find linorobot2_description)/urdf/sensors/depth_sensor.urdf.xacro" />
   <xacro:include filename="$(find linorobot2_description)/urdf/controllers/omni_drive.urdf.xacro" />
   <xacro:base
@@ -55,4 +56,7 @@
     <xacro:insert_block name="laser_pose" />
   </xacro:ld06>
+  <xacro:depth_sensor>
+    <xacro:insert_block name="depth_sensor_pose" />
+  </xacro:depth_sensor>
   <xacro:omni_drive_controller/>
 </robot>

Commit message: fixed robot wheels

File: linorobot2_description/urdf/2wd_properties.urdf.xacro (robot description, xacro)
@@ -7,11 +7,11 @@
   <xacro:property name="wheel_radius" value="0.045" />
   <xacro:property name="wheel_width" value="0.01" />
-  <xacro:property name="wheel_pos_x" value="-0.0415" />
+  <xacro:property name="wheel_pos_x" value="0.0415" />
   <xacro:property name="wheel_pos_y" value="0.1" />
   <xacro:property name="wheel_pos_z" value="0.023" />
   <xacro:property name="wheel_mass" value=".1" />
   <xacro:property name="wheel_torque" value="20" />
-  <xacro:property name="front_caster_wheel" value="true" />
-  <xacro:property name="rear_caster_wheel" value="false" />
+  <xacro:property name="front_caster_wheel" value="false" />
+  <xacro:property name="rear_caster_wheel" value="true" />
   <xacro:property name="laser_pose">
     <origin xyz="0 0 0.1" rpy="0 0 0"/>

Commit message: updated properties

File: linorobot2_description/urdf/2wd_properties.urdf.xacro (robot description, xacro)
@@ -1,19 +1,19 @@
 <?xml version="1.0"?>
 <robot xmlns:xacro="http://ros.org/wiki/xacro">
-  <xacro:property name="base_length" value="0.17" />
-  <xacro:property name="base_width" value="0.17" />
+  <xacro:property name="base_length" value="0.24" />
+  <xacro:property name="base_width" value="0.22" />
   <xacro:property name="base_height" value="0.003" />
   <xacro:property name="base_mass" value="1" />
   <xacro:property name="wheel_radius" value="0.045" />
   <xacro:property name="wheel_width" value="0.01" />
-  <xacro:property name="wheel_pos_x" value="0.0415" />
-  <xacro:property name="wheel_pos_y" value="0.1" />
+  <xacro:property name="wheel_pos_x" value="0.0" />
+  <xacro:property name="wheel_pos_y" value="0.13" />
   <xacro:property name="wheel_pos_z" value="0.023" />
   <xacro:property name="wheel_mass" value=".1" />
   <xacro:property name="wheel_torque" value="20" />
-  <xacro:property name="front_caster_wheel" value="false" />
+  <xacro:property name="front_caster_wheel" value="true" />
   <xacro:property name="rear_caster_wheel" value="true" />
   <xacro:property name="laser_pose">
-    <origin xyz="0 0 0.1" rpy="0 0 0"/>
+    <origin xyz="0.12 0 0.1" rpy="0 0 0"/>
   </xacro:property>
   <xacro:property name="depth_sensor_pose">

Commit message: updated prototype robot

File: linorobot2_description/urdf/2wd_properties.urdf.xacro (robot description, xacro)
@@ -2,5 +2,5 @@
 <robot xmlns:xacro="http://ros.org/wiki/xacro">
   <xacro:property name="base_length" value="0.24" />
-  <xacro:property name="base_width" value="0.22" />
+  <xacro:property name="base_width" value="0.275" />
   <xacro:property name="base_height" value="0.003" />
   <xacro:property name="base_mass" value="1" />
@@ -9,5 +9,5 @@
   <xacro:property name="wheel_pos_x" value="0.0" />
   <xacro:property name="wheel_pos_y" value="0.13" />
-  <xacro:property name="wheel_pos_z" value="0.023" />
+  <xacro:property name="wheel_pos_z" value="-0.03" />
   <xacro:property name="wheel_mass" value=".1" />
   <xacro:property name="wheel_torque" value="20" />
@@ -15,8 +15,8 @@
   <xacro:property name="rear_caster_wheel" value="true" />
   <xacro:property name="laser_pose">
-    <origin xyz="0.12 0 0.1" rpy="0 0 0"/>
+    <origin xyz="0.12 0 0.33" rpy="0 0 0"/>
   </xacro:property>
   <xacro:property name="depth_sensor_pose">
-    <origin xyz="0.085 0 0.02" rpy="0 0 0"/>
+    <origin xyz="0.14 0 0.26" rpy="0 0 0"/>
   </xacro:property>
 </robot>

Commit message: updated robot prototype

File: linorobot2_description/urdf/2wd_properties.urdf.xacro (robot description, xacro)
@@ -18,5 +18,5 @@
   </xacro:property>
   <xacro:property name="depth_sensor_pose">
-    <origin xyz="0.14 0 0.26" rpy="0 0 0"/>
+    <origin xyz="0.14 -0.03 0.065" rpy="-1.57 0 0"/>
   </xacro:property>
 </robot>

Commit message: updated depth sensor position

File: linorobot2_description/urdf/2wd_properties.urdf.xacro (robot description, xacro)
@@ -18,5 +18,5 @@
   </xacro:property>
   <xacro:property name="depth_sensor_pose">
-    <origin xyz="0.14 -0.03 0.065" rpy="-1.57 0 0"/>
+    <origin xyz="0.1 0.0 0.255" rpy="3.1416 0.349066 0"/>
   </xacro:property>
 </robot>

Commit message: updated sensor pose

File: linorobot2_description/urdf/2wd_properties.urdf.xacro (robot description, xacro)
@@ -18,5 +18,5 @@
   </xacro:property>
   <xacro:property name="depth_sensor_pose">
-    <origin xyz="0.1 0.0 0.255" rpy="3.1416 0.349066 0"/>
+    <origin xyz="0.14 0.0 0.045" rpy="0 0 0"/>
   </xacro:property>
 </robot>

Commit message: camera urdf

File: linorobot2_description/urdf/2wd_properties.urdf.xacro (robot description, xacro)
@@ -1,22 +1,31 @@
 <?xml version="1.0"?>
 <robot xmlns:xacro="http://ros.org/wiki/xacro">
-  <xacro:property name="base_length" value="0.24" />
-  <xacro:property name="base_width" value="0.275" />
-  <xacro:property name="base_height" value="0.003" />
+  <xacro:property name="base_length" value="0.50" />
+  <xacro:property name="base_width" value="0.40" />
+  <xacro:property name="base_height" value="0.20" />
   <xacro:property name="base_mass" value="1" />
-  <xacro:property name="wheel_radius" value="0.045" />
-  <xacro:property name="wheel_width" value="0.01" />
-  <xacro:property name="wheel_pos_x" value="0.0" />
-  <xacro:property name="wheel_pos_y" value="0.13" />
-  <xacro:property name="wheel_pos_z" value="-0.03" />
-  <xacro:property name="wheel_mass" value=".1" />
+  <xacro:property name="wheel_radius" value="0.08255" />
+  <xacro:property name="wheel_width" value="0.058" />
+  <xacro:property name="wheel_pos_x" value="0.15" />
+  <xacro:property name="wheel_pos_y" value="0.25" />
+  <xacro:property name="wheel_pos_z" value="-0.08255" />
+  <xacro:property name="wheel_mass" value="3" />
   <xacro:property name="wheel_torque" value="20" />
-  <xacro:property name="front_caster_wheel" value="true" />
-  <xacro:property name="rear_caster_wheel" value="true" />
+  <!-- <xacro:property name="front_caster_wheel" value="true" />
+  <xacro:property name="rear_caster_wheel" value="true" /> -->
+  <xacro:property name="lift_plate_length" value="0.30" />
+  <xacro:property name="lift_plate_width" value="0.30" />
+  <xacro:property name="lift_plate_height" value="0.01" />
+  <xacro:property name="lift_plate_mass" value="0.5" />
+  <xacro:property name="lift_plate_wheel_pos_x" value="-0.1" />
+  <xacro:property name="lift_plate_wheel_pos_y" value="0" />
+  <xacro:property name="lift_plate_wheel_pos_z" value="0.35" />
+  <xacro:property name="caster_wheel_x" value="-0.15" />
+  <xacro:property name="caster_wheel_y" value="0.15" />
   <xacro:property name="laser_pose">
-    <origin xyz="0.12 0 0.33" rpy="0 0 0"/>
+    <origin xyz="0.12 0 0.15" rpy="0 0 0"/>
   </xacro:property>
   <xacro:property name="depth_sensor_pose">
-    <origin xyz="0.14 0.0 0.045" rpy="0 0 0"/>
+    <origin xyz="0.3 0.0 0.045" rpy="0 0 0"/>
   </xacro:property>
 </robot>

Commit message: added lidar

File: linorobot2_description/urdf/2wd_properties.urdf.xacro (robot description, xacro)
@@ -1,7 +1,7 @@
 <?xml version="1.0"?>
 <robot xmlns:xacro="http://ros.org/wiki/xacro">
-  <xacro:property name="base_length" value="0.50" />
+  <xacro:property name="base_length" value="0.60" />
   <xacro:property name="base_width" value="0.40" />
-  <xacro:property name="base_height" value="0.20" />
+  <xacro:property name="base_height" value="0.30" />
   <xacro:property name="base_mass" value="1" />
   <xacro:property name="wheel_radius" value="0.08255" />

File: linorobot2_description/urdf/robots/LeoGV.urdf.xacro (robot description, xacro)
@@ -2,11 +2,12 @@
 <robot name="LeoGV" xmlns:xacro="http://ros.org/wiki/xacro">
   <xacro:include filename="$(find linorobot2_description)/urdf/2wd_properties.urdf.xacro" />
+  <!-- <xacro:include filename="$(find linorobot2_description)/urdf/inertial_macros.xacro" /> -->
   <xacro:include filename="$(find linorobot2_description)/urdf/mech/base.urdf.xacro" />
   <xacro:include filename="$(find linorobot2_description)/urdf/mech/lift_plate_LeoGV.urdf.xacro" />
   <xacro:include filename="$(find linorobot2_description)/urdf/mech/wheel.urdf.xacro" />
   <xacro:include filename="$(find linorobot2_description)/urdf/mech/caster_wheel_LeoGV.urdf.xacro" />
-  <xacro:include filename="$(find linorobot2_description)/urdf/sensors/imu.urdf.xacro" />
+  <!-- <xacro:include filename="$(find linorobot2_description)/urdf/sensors/imu.urdf.xacro" /> -->
   <xacro:include filename="$(find linorobot2_description)/urdf/sensors/generic_laser.urdf.xacro" />
-  <xacro:include filename="$(find linorobot2_description)/urdf/sensors/depth_sensor.urdf.xacro" />
+  <!-- <xacro:include filename="$(find linorobot2_description)/urdf/sensors/depth_sensor.urdf.xacro" /> -->
   <xacro:include filename="$(find linorobot2_description)/urdf/sensors/camera_LeoGV.urdf.xacro" />
   <xacro:include filename="$(find linorobot2_description)/urdf/controllers/diff_drive.urdf.xacro" />

File: linorobot2_description/urdf/sensors/camera_LeoGV.urdf.xacro (robot description, xacro)
@@ -1,4 +1,3 @@
 <robot xmlns:xacro="http://ros.org/wiki/xacro">
-  <xacro:property name="M_PI" value="3.1415926535897931" />
   <xacro:macro name="camera_LeoGV" params="*origin">
     <!-- camera_link describes the camera at the end of the arm -->
@@ -61,5 +60,5 @@
         <update_rate>5</update_rate>
         <camera name="camera">
-          <horizontal_fov>1.50098</horizontal_fov>
+          <horizontal_fov>1.089</horizontal_fov>
           <image>
             <width>640</width>
@@ -68,20 +67,20 @@
           </image>
           <clip>
-              <near>0.02</near>
-              <far>300</far>
+              <near>0.05</near>
+              <far>8.0</far>
           </clip>
-          <noise>
+          <!-- <noise>
               <type>gaussian</type>
               <mean>0.0</mean>
               <stddev>0.007</stddev>
-          </noise>
+          </noise>           -->
         </camera>
         <plugin name="camera_controller" filename="libgazebo_ros_camera.so">
           <ros>
-            <remapping>/camera/camera_info:=/camera/color/camera_info</remapping>
-            <remapping>/camera/image_raw:=/camera/color/image_raw</remapping>
-            <remapping>/camera/points:=/camera/depth/color/points</remapping>
-            <remapping>/camera/depth/image_raw:=/camera/depth/image_rect_raw</remapping>
-            <qos>
+            <!-- <remapping>/camera/camera_info:=/camera/color/camera_info</remapping>
+            <remapping>/camera/image_raw:=/camera/color/image_raw</remapping> -->
+            <!-- <remapping>/camera/points:=/camera/depth/color/points</remapping>
+            <remapping>/camera/depth/image_raw:=/camera/depth/image_rect_raw</remapping> -->
+            <!-- <qos>
               <topic name="/camera/depth/color/points">
                 <publisher>
@@ -89,15 +88,15 @@
                 </publisher>
               </topic>
-            </qos>
+            </qos> -->
           </ros>
-          <min_depth>0.015</min_depth>
+          <!-- <min_depth>0.015</min_depth>
           <max_depth>3.0</max_depth>
-          <hack_baseline>0.07</hack_baseline>
+          <hack_baseline>0.07</hack_baseline> -->
           <frame_name>camera_link_optical</frame_name>
-          <distortion_k1>0.00000001</distortion_k1>
+          <!-- <distortion_k1>0.00000001</distortion_k1>
           <distortion_k2>0.00000001</distortion_k2>
           <distortion_k3>0.00000001</distortion_k3>
           <distortion_t1>0.00000001</distortion_t1>
-          <distortion_t2>0.00000001</distortion_t2>
+          <distortion_t2>0.00000001</distortion_t2> -->
         </plugin>
       </sensor>

File: linorobot2_description/urdf/sensors/generic_laser.urdf.xacro (robot description, xacro)
@@ -3,30 +3,61 @@
   <xacro:include filename="$(find linorobot2_description)/urdf/sensors/laser.urdf.xacro" />
   <xacro:macro name="generic_laser" params="*origin">
-    <xacro:laser
-      update_rate="10"
-      ray_count="360"
-      min_angle="-3.1416"
-      max_angle="3.1416"
-      min_range="0.08"
-      max_range="12.0"
-      frame_id="laser"
-      topic_name="scan"
-    >
-      <xacro:insert_block name="origin" />
-    </xacro:laser>
-  </xacro:macro>
-  <xacro:macro name="generic_base_laser" params="*origin">
-    <xacro:laser
-      update_rate="10"
-      ray_count="360"
-      min_angle="-3.1416"
-      max_angle="3.1416"
-      min_range="0.21"
-      max_range="5.5"
-      frame_id="base_laser"
-      topic_name="base/scan"
-    >
-      <xacro:insert_block name="origin" />
-    </xacro:laser>
-  </xacro:macro>
+    <link name="laser_frame">
+        <visual>
+            <geometry>
+                <cylinder radius="0.05" length="0.04"/>
+            </geometry>
+            <material name="black"/>
+        </visual>
+        <visual>
+            <origin xyz="0 0 -0.05"/>
+            <geometry>
+                <cylinder radius="0.01" length="0.1"/>
+            </geometry>
+            <material name="black"/>
+        </visual>
+        <collision>
+            <geometry>
+                <cylinder radius="0.05" length="0.04"/>
+            </geometry>
+        </collision>
+        <!-- <xacro:inertial_cylinder mass="0.1" length="0.04" radius="0.05">
+            <origin xyz="0 0 0" rpy="0 0 0"/> -->
+        <!-- </xacro:inertial_cylinder> -->
+    </link>
+    <joint name="laser_joint" type="fixed">
+        <parent link="base_link"/>
+        <child link="laser_frame"/>
+        <!-- <origin xyz="0.1 0 0.175" rpy="0 0 0"/> -->
+        <xacro:insert_block name="origin" />
+    </joint>
+    <gazebo reference="laser_frame">
+        <material>Gazebo/Black</material>
+        <sensor name="laser" type="ray">
+            <pose> 0 0 0 0 0 0 </pose>
+            <visualize>false</visualize>
+            <update_rate>10</update_rate>
+            <ray>
+                <scan>
+                    <horizontal>
+                        <samples>360</samples>
+                        <min_angle>-3.14</min_angle>
+                        <max_angle>3.14</max_angle>
+                    </horizontal>
+                </scan>
+                <range>
+                    <min>0.3</min>
+                    <max>12</max>
+                </range>
+            </ray>
+            <plugin name="laser_controller" filename="libgazebo_ros_ray_sensor.so">
+                <ros>
+                    <argument>~/out:=scan</argument>
+                </ros>
+                <output_type>sensor_msgs/LaserScan</output_type>
+                <frame_name>laser_frame</frame_name>
+            </plugin>
+        </sensor>
+    </gazebo>
+</xacro:macro>
 </robot>

Commit message: amazon warehouse working

File: linorobot2_description/urdf/2wd_properties.urdf.xacro (robot description, xacro)
@@ -9,5 +9,5 @@
   <xacro:property name="wheel_pos_x" value="0.15" />
   <xacro:property name="wheel_pos_y" value="0.25" />
-  <xacro:property name="wheel_pos_z" value="-0.08255" />
+  <xacro:property name="wheel_pos_z" value="0.08255" />
   <xacro:property name="wheel_mass" value="3" />
   <xacro:property name="wheel_torque" value="20" />

File: linorobot2_description/urdf/robots/LeoGV.urdf.xacro (robot description, xacro)
@@ -35,5 +35,5 @@
     pos_x="${wheel_pos_x}"
     pos_y="${wheel_pos_y}"
-    pos_z="${wheel_pos_z}"
+    pos_z="${-base_height/2}"
     mass="${wheel_mass}"
   />
@@ -44,5 +44,5 @@
     pos_x="${wheel_pos_x}"
     pos_y="${-wheel_pos_y}"
-    pos_z="${wheel_pos_z}"
+    pos_z="${-base_height/2}"
     mass="${wheel_mass}"
   />
@@ -50,5 +50,5 @@
     side="left"
     wheel_radius="${wheel_radius}"
-    wheel_pos_z="${wheel_pos_z}"
+    wheel_pos_z="${base_height/2}"
     caster_wheel_x="${caster_wheel_x}"
     caster_wheel_y="${caster_wheel_y}"
@@ -58,5 +58,5 @@
     side="right"
     wheel_radius="${wheel_radius}"
-    wheel_pos_z="${wheel_pos_z}"
+    wheel_pos_z="${base_height/2}"
     caster_wheel_x="${caster_wheel_x}"
     caster_wheel_y="${-caster_wheel_y}"
