Commit message: added mesh files, and updated the plugin for 4wd and mecanum

File: linorobot2_description/urdf/2wd_properties.urdf.xacro (robot description, xacro)
@@ -1,10 +1,13 @@
 <?xml version="1.0"?>
 <robot xmlns:xacro="http://ros.org/wiki/xacro">
-  <xacro:property name="base_length" value="0.24" />
-  <xacro:property name="base_width" value="0.275" />
-  <xacro:property name="base_height" value="0.003" />
+  <xacro:property name="base_length" value="0.27" />
+  <xacro:property name="base_width" value="0.27" />
+  <xacro:property name="base_height" value="0.09" />
   <xacro:property name="base_mass" value="1" />
-  <xacro:property name="wheel_radius" value="0.045" />
-  <xacro:property name="wheel_width" value="0.01" />
+  <!-- set empty on the wheel_mesh_file to use geometry instead of mesh -->
+  <xacro:property name="base_mesh_file" value="" />
+  <!-- <xacro:property name="base_mesh_file" value="file://$(find linorobot2_description)/meshes/base.dae" /> -->
+  <xacro:property name="wheel_radius" value="0.033" />
+  <xacro:property name="wheel_width" value="0.018" />
   <xacro:property name="wheel_pos_x" value="0.0" />
   <xacro:property name="wheel_pos_y" value="0.145" />
@@ -14,6 +17,9 @@
   <xacro:property name="front_caster_wheel" value="true" />
   <xacro:property name="rear_caster_wheel" value="true" />
+  <!-- set empty on the wheel_mesh_file to use geometry instead of mesh -->
+  <xacro:property name="wheel_mesh_file" value="" />
+  <!-- <xacro:property name="wheel_mesh_file" value="file://$(find linorobot2_description)/meshes/tire.dae" /> -->
   <xacro:property name="laser_pose">
-    <origin xyz="0.12 0 0.33" rpy="0 0 0"/>
+    <origin xyz="0.0 0 0.17" rpy="0 0 0"/>
   </xacro:property>
   <xacro:property name="depth_sensor_pose">

File: linorobot2_description/urdf/4wd_properties.urdf.xacro (robot description, xacro)
@@ -1,10 +1,13 @@
 <?xml version="1.0"?>
 <robot xmlns:xacro="http://ros.org/wiki/xacro">
-  <xacro:property name="base_length" value="0.445" />
-  <xacro:property name="base_width" value="0.200" />
-  <xacro:property name="base_height" value="0.129" />
-  <xacro:property name="base_mass" value="10" />
-  <xacro:property name="wheel_radius" value="0.07162" />
-  <xacro:property name="wheel_width" value="0.05" />
+  <xacro:property name="base_length" value="0.27" />
+  <xacro:property name="base_width" value="0.27" />
+  <xacro:property name="base_height" value="0.09" />
+  <xacro:property name="base_mass" value="1" />
+  <!-- set empty on the wheel_mesh_file to use geometry instead of mesh -->
+  <xacro:property name="base_mesh_file" value="" />
+  <!-- <xacro:property name="base_mesh_file" value="file://$(find linorobot2_description)/meshes/base.dae" /> -->
+  <xacro:property name="wheel_radius" value="0.033" />
+  <xacro:property name="wheel_width" value="0.018" />
   <xacro:property name="wheel_pos_x" value="0.120" />
   <xacro:property name="wheel_pos_y" value="0.1355" />
@@ -12,4 +15,7 @@
   <xacro:property name="wheel_mass" value=".6" />
   <xacro:property name="wheel_torque" value="20" />
+  <!-- set empty on the wheel_mesh_file to use geometry instead of mesh -->
+  <xacro:property name="wheel_mesh_file" value="" />
+  <!-- <xacro:property name="wheel_mesh_file" value="file://$(find linorobot2_description)/meshes/tire.dae" /> -->
   <xacro:property name="laser_pose">
     <origin xyz="-0.0475 0 0.125" rpy="0 0 0"/>

File: linorobot2_description/urdf/controllers/diff_drive.urdf.xacro (robot description, xacro)
@@ -2,4 +2,7 @@
   <xacro:macro name="diff_drive_controller" params="wheel_separation wheel_radius">
     <gazebo>
+      <!-- <plugin
+        filename="ignition-gazebo-diff-drive-system"
+        name="ignition::gazebo::systems::DiffDrive"> -->
       <plugin
         filename="gz-sim-diff-drive-system"

File: linorobot2_description/urdf/controllers/omni_drive.urdf.xacro (robot description, xacro)
@@ -9,4 +9,5 @@
         <child_frame_id>base_footprint</child_frame_id>
         <odom_topic>odom/unfiltered</odom_topic>
+        <tf_topic>/tf</tf_topic>
         <front_left_joint>front_left_wheel_joint</front_left_joint>
         <front_right_joint>front_right_wheel_joint</front_right_joint>
@@ -17,6 +18,19 @@
         <wheel_radius>${wheel_radius}</wheel_radius>
         <odom_publish_frequency>50</odom_publish_frequency>
+        <min_acceleration>-5</min_acceleration>
+        <max_acceleration>5</max_acceleration>
       </plugin>
-  </gazebo>
+    </gazebo>
+    <gazebo>
+      <plugin filename="gz-sim-joint-state-publisher-system"
+        name="gz::sim::systems::JointStatePublisher">
+        <topic>joint_states</topic>
+        <update_rate>30</update_rate>
+        <joint_name>front_left_wheel_joint</joint_name>
+        <joint_name>front_right_wheel_joint</joint_name>
+        <joint_name>rear_left_wheel_joint</joint_name>
+        <joint_name>rear_right_wheel_joint</joint_name>
+      </plugin>
+    </gazebo>
   </xacro:macro>
 </robot>

File: linorobot2_description/urdf/controllers/skid_steer.urdf.xacro (robot description, xacro)
@@ -2,18 +2,34 @@
   <xacro:macro name="diff_drive_controller" params="wheel_separation wheel_radius">
     <gazebo>
+      <!-- <plugin
+        filename="ignition-gazebo-diff-drive-system"
+        name="ignition::gazebo::systems::DiffDrive"> -->
       <plugin
-        filename="ignition-gazebo-diff-drive-system"
-        name="ignition::gazebo::systems::DiffDrive">
-        <topic>/cmd_vel</topic>
-        <frame_id>odom</frame_id>
-        <child_frame_id>base_footprint</child_frame_id>
-        <odom_topic>odom/unfiltered</odom_topic>
-        <left_joint>front_left_wheel_joint</left_joint>
-        <right_joint>front_right_wheel_joint</right_joint>
-        <left_joint>rear_left_wheel_joint</left_joint>
-        <right_joint>rear_right_wheel_joint</right_joint>
-        <wheel_separation>${wheel_separation}</wheel_separation>
-        <wheel_radius>${wheel_radius}</wheel_radius>
-        <odom_publish_frequency>50</odom_publish_frequency>
+        filename="gz-sim-diff-drive-system"
+        name="gz::sim::systems::DiffDrive">
+          <topic>/cmd_vel</topic>
+          <frame_id>odom</frame_id>
+          <child_frame_id>base_footprint</child_frame_id>
+          <odom_topic>odom/unfiltered</odom_topic>
+          <tf_topic>/tf</tf_topic>
+          <max_linear_acceleration>1.0</max_linear_acceleration>
+          <left_joint>front_left_wheel_joint</left_joint>
+          <right_joint>front_right_wheel_joint</right_joint>
+          <left_joint>rear_left_wheel_joint</left_joint>
+          <right_joint>rear_right_wheel_joint</right_joint>
+          <wheel_separation>${wheel_separation}</wheel_separation>
+          <wheel_radius>${wheel_radius}</wheel_radius>
+          <odom_publish_frequency>50</odom_publish_frequency>
+      </plugin>
+    </gazebo>
+    <gazebo>
+      <plugin filename="gz-sim-joint-state-publisher-system"
+        name="gz::sim::systems::JointStatePublisher">
+        <topic>joint_states</topic>
+        <update_rate>30</update_rate>
+        <joint_name>front_left_wheel_joint</joint_name>
+        <joint_name>front_right_wheel_joint</joint_name>
+        <joint_name>rear_left_wheel_joint</joint_name>
+        <joint_name>rear_right_wheel_joint</joint_name>
       </plugin>
     </gazebo>

File: linorobot2_description/urdf/mecanum_properties.urdf.xacro (robot description, xacro)
@@ -1,10 +1,13 @@
 <?xml version="1.0"?>
 <robot xmlns:xacro="http://ros.org/wiki/xacro">
-  <xacro:property name="base_length" value="0.445" />
-  <xacro:property name="base_width" value="0.200" />
-  <xacro:property name="base_height" value="0.129" />
-  <xacro:property name="base_mass" value="10" />
-  <xacro:property name="wheel_radius" value="0.07162" />
-  <xacro:property name="wheel_width" value="0.05" />
+  <xacro:property name="base_length" value="0.27" />
+  <xacro:property name="base_width" value="0.27" />
+  <xacro:property name="base_height" value="0.09" />
+  <xacro:property name="base_mass" value="1" />
+  <!-- set empty on the wheel_mesh_file to use geometry instead of mesh -->
+  <xacro:property name="base_mesh_file" value="" />
+  <!-- <xacro:property name="base_mesh_file" value="file://$(find linorobot2_description)/meshes/base.dae" /> -->
+  <xacro:property name="wheel_radius" value="0.033" />
+  <xacro:property name="wheel_width" value="0.018" />
   <xacro:property name="wheel_pos_x" value="0.120" />
   <xacro:property name="wheel_pos_y" value="0.1355" />
@@ -12,4 +15,7 @@
   <xacro:property name="wheel_mass" value=".6" />
   <xacro:property name="wheel_torque" value="20" />
+  <!-- set empty on the wheel_mesh_file to use geometry instead of mesh -->
+  <xacro:property name="wheel_mesh_file" value="" />
+  <!-- <xacro:property name="wheel_mesh_file" value="file://$(find linorobot2_description)/meshes/tire.dae" /> -->
   <xacro:property name="laser_pose">
     <origin xyz="-0.0475 0 0.125" rpy="0 0 0"/>

File: linorobot2_description/urdf/mech/base.urdf.xacro (robot description, xacro)
@@ -1,5 +1,5 @@
 <?xml version="1.0"?>
 <robot xmlns:xacro="http://ros.org/wiki/xacro">
-  <xacro:macro name="base" params="length width height mass wheel_radius wheel_pos_z">
+  <xacro:macro name="base" params="length width height mass wheel_radius wheel_pos_z mesh_file">
     <link name="base_footprint"/>
     <link name="base_link">
@@ -7,6 +7,10 @@
         <origin xyz="0 0 0" rpy="0 0 0"/>
         <geometry>
-          <box size="${length} ${width} ${height}"/>
-          <!-- <mesh filename="" scale="0.001 0.001 0.001"/> -->
+          <xacro:if value="${mesh_file == ''}">
+            <box size="${length} ${width} ${height}"/>
+          </xacro:if>
+          <xacro:unless value="${mesh_file == ''}">
+            <mesh filename="${mesh_file}" scale="1 1 1"/>
+          </xacro:unless>
         </geometry>
         <material name="yellow">

File: linorobot2_description/urdf/mech/mecanum_wheel.urdf.xacro (robot description, xacro)
@@ -1,10 +1,15 @@
 <?xml version="1.0"?>
 <robot xmlns:xacro="http://ros.org/wiki/xacro">
-  <xacro:macro name="mecanum_wheel" params="side radius width pos_x pos_y pos_z mass">
+  <xacro:macro name="mecanum_wheel" params="side radius width pos_x pos_y pos_z mass mesh_file">
     <link name="${side}_wheel_link">
       <visual>
         <origin xyz="0 0 0" rpy="${pi/2} 0 0"/>
         <geometry>
-          <cylinder radius="${radius}" length="${width}"/>
+          <xacro:if value="${mesh_file == ''}">
+            <cylinder radius="${radius}" length="${width}"/>
+          </xacro:if>
+          <xacro:unless value="${mesh_file == ''}">
+            <mesh filename="${mesh_file}" scale="1 1 1"/>
+          </xacro:unless>
         </geometry>
         <material name="blue">
@@ -15,5 +20,6 @@
         <origin xyz="0 0 0" rpy="${pi/2} 0 0"/>
         <geometry>
-          <cylinder radius="${radius}" length="${width}"/>
+          <sphere radius="${radius}"/>
+          <!-- <cylinder radius="${radius}" length="${width}"/> -->
         </geometry>
       </collision>

File: linorobot2_description/urdf/mech/wheel.urdf.xacro (robot description, xacro)
@@ -1,10 +1,15 @@
 <?xml version="1.0"?>
 <robot xmlns:xacro="http://ros.org/wiki/xacro">
-  <xacro:macro name="wheel" params="side radius width pos_x pos_y pos_z mass">
+  <xacro:macro name="wheel" params="side radius width pos_x pos_y pos_z mass mesh_file">
     <link name="${side}_wheel_link">
       <visual>
         <origin xyz="0 0 0" rpy="${pi/2} 0 0"/>
         <geometry>
-          <cylinder radius="${radius}" length="${width}"/>
+          <xacro:if value="${mesh_file == ''}">
+            <cylinder radius="${radius}" length="${width}"/>
+          </xacro:if>
+          <xacro:unless value="${mesh_file == ''}">
+            <mesh filename="${mesh_file}" scale="1 1 1"/>
+          </xacro:unless>
         </geometry>
         <material name="blue">

File: linorobot2_description/urdf/robots/2wd.urdf.xacro (robot description, xacro)
@@ -18,5 +18,6 @@
     wheel_radius="${wheel_radius}"
     wheel_pos_z="${wheel_pos_z}"
-/>
+    mesh_file="${base_mesh_file}"
+  />
   <xacro:wheel
     side="left"
@@ -27,4 +28,5 @@
     pos_z="${wheel_pos_z}"
     mass="${wheel_mass}"
+    mesh_file="${wheel_mesh_file}"
   />
   <xacro:wheel
@@ -36,4 +38,5 @@
     pos_z="${wheel_pos_z}"
     mass="${wheel_mass}"
+    mesh_file="${wheel_mesh_file}"
   />
   <xacro:if value="${front_caster_wheel}">

File: linorobot2_description/urdf/robots/4wd.urdf.xacro (robot description, xacro)
@@ -1,4 +1,4 @@
 <?xml version="1.0"?>
-<robot name="linorobot2_2wd" xmlns:xacro="http://ros.org/wiki/xacro">
+<robot name="linorobot2_4wd" xmlns:xacro="http://ros.org/wiki/xacro">
   <xacro:arg name="sim" default="false" />
   <xacro:include filename="$(find linorobot2_description)/urdf/4wd_properties.urdf.xacro" />
@@ -17,5 +17,6 @@
     wheel_radius="${wheel_radius}"
     wheel_pos_z="${wheel_pos_z}"
-/>
+    mesh_file="${base_mesh_file}"
+  />
   <xacro:wheel
     side="front_left"
@@ -26,4 +27,5 @@
     pos_z="${wheel_pos_z}"
     mass="${wheel_mass}"
+    mesh_file="${wheel_mesh_file}"
   />
   <xacro:wheel
@@ -35,4 +37,5 @@
     pos_z="${wheel_pos_z}"
     mass="${wheel_mass}"
+    mesh_file="${wheel_mesh_file}"
   />
   <xacro:wheel
@@ -44,4 +47,5 @@
     pos_z="${wheel_pos_z}"
     mass="${wheel_mass}"
+    mesh_file="${wheel_mesh_file}"
   />
   <xacro:wheel
@@ -53,4 +57,5 @@
     pos_z="${wheel_pos_z}"
     mass="${wheel_mass}"
+    mesh_file="${wheel_mesh_file}"
   />
   <xacro:imu/>

File: linorobot2_description/urdf/robots/mecanum.urdf.xacro (robot description, xacro)
@@ -1,4 +1,4 @@
 <?xml version="1.0"?>
-<robot name="linorobot2_2wd" xmlns:xacro="http://ros.org/wiki/xacro">
+<robot name="linorobot2_mecanum" xmlns:xacro="http://ros.org/wiki/xacro">
   <xacro:arg name="sim" default="false" />
   <xacro:include filename="$(find linorobot2_description)/urdf/mecanum_properties.urdf.xacro" />
@@ -17,5 +17,6 @@
     wheel_radius="${wheel_radius}"
     wheel_pos_z="${wheel_pos_z}"
-/>
+    mesh_file="${base_mesh_file}"
+  />
   <xacro:mecanum_wheel
     side="front_left"
@@ -26,4 +27,5 @@
     pos_z="${wheel_pos_z}"
     mass="${wheel_mass}"
+    mesh_file="${wheel_mesh_file}"
   />
   <xacro:mecanum_wheel
@@ -35,4 +37,5 @@
     pos_z="${wheel_pos_z}"
     mass="${wheel_mass}"
+    mesh_file="${wheel_mesh_file}"
   />
   <xacro:mecanum_wheel
@@ -44,4 +47,5 @@
     pos_z="${wheel_pos_z}"
     mass="${wheel_mass}"
+    mesh_file="${wheel_mesh_file}"
   />
   <xacro:mecanum_wheel
@@ -53,4 +57,5 @@
     pos_z="${wheel_pos_z}"
     mass="${wheel_mass}"
+    mesh_file="${wheel_mesh_file}"
   />
   <xacro:imu/>

Commit message: revert properties values

File: linorobot2_description/urdf/2wd_properties.urdf.xacro (robot description, xacro)
@@ -1,15 +1,15 @@
 <?xml version="1.0"?>
 <robot xmlns:xacro="http://ros.org/wiki/xacro">
-  <xacro:property name="base_length" value="0.27" />
-  <xacro:property name="base_width" value="0.27" />
-  <xacro:property name="base_height" value="0.09" />
+  <xacro:property name="base_length" value="0.24" />
+  <xacro:property name="base_width" value="0.275" />
+  <xacro:property name="base_height" value="0.003" />
   <xacro:property name="base_mass" value="1" />
   <!-- set empty on the wheel_mesh_file to use geometry instead of mesh -->
   <xacro:property name="base_mesh_file" value="" />
   <!-- <xacro:property name="base_mesh_file" value="file://$(find linorobot2_description)/meshes/base.dae" /> -->
-  <xacro:property name="wheel_radius" value="0.033" />
-  <xacro:property name="wheel_width" value="0.018" />
+  <xacro:property name="wheel_radius" value="0.045" />
+  <xacro:property name="wheel_width" value="0.01" />
   <xacro:property name="wheel_pos_x" value="0.0" />
-  <xacro:property name="wheel_pos_y" value="0.145" />
+  <xacro:property name="wheel_pos_y" value="0.13" />
   <xacro:property name="wheel_pos_z" value="-0.03" />
   <xacro:property name="wheel_mass" value=".1" />

File: linorobot2_description/urdf/4wd_properties.urdf.xacro (robot description, xacro)
@@ -1,13 +1,13 @@
 <?xml version="1.0"?>
 <robot xmlns:xacro="http://ros.org/wiki/xacro">
-  <xacro:property name="base_length" value="0.27" />
-  <xacro:property name="base_width" value="0.27" />
-  <xacro:property name="base_height" value="0.09" />
-  <xacro:property name="base_mass" value="1" />
+  <xacro:property name="base_length" value="0.445" />
+  <xacro:property name="base_width" value="0.200" />
+  <xacro:property name="base_height" value="0.129" />
+  <xacro:property name="base_mass" value="10" />
   <!-- set empty on the wheel_mesh_file to use geometry instead of mesh -->
   <xacro:property name="base_mesh_file" value="" />
   <!-- <xacro:property name="base_mesh_file" value="file://$(find linorobot2_description)/meshes/base.dae" /> -->
-  <xacro:property name="wheel_radius" value="0.033" />
-  <xacro:property name="wheel_width" value="0.018" />
+  <xacro:property name="wheel_radius" value="0.07162" />
+  <xacro:property name="wheel_width" value="0.05" />
   <xacro:property name="wheel_pos_x" value="0.120" />
   <xacro:property name="wheel_pos_y" value="0.1355" />

File: linorobot2_description/urdf/mecanum_properties.urdf.xacro (robot description, xacro)
@@ -1,13 +1,13 @@
 <?xml version="1.0"?>
 <robot xmlns:xacro="http://ros.org/wiki/xacro">
-  <xacro:property name="base_length" value="0.27" />
-  <xacro:property name="base_width" value="0.27" />
-  <xacro:property name="base_height" value="0.09" />
-  <xacro:property name="base_mass" value="1" />
+  <xacro:property name="base_length" value="0.445" />
+  <xacro:property name="base_width" value="0.200" />
+  <xacro:property name="base_height" value="0.129" />
+  <xacro:property name="base_mass" value="10" />
   <!-- set empty on the wheel_mesh_file to use geometry instead of mesh -->
   <xacro:property name="base_mesh_file" value="" />
   <!-- <xacro:property name="base_mesh_file" value="file://$(find linorobot2_description)/meshes/base.dae" /> -->
-  <xacro:property name="wheel_radius" value="0.033" />
-  <xacro:property name="wheel_width" value="0.018" />
+  <xacro:property name="wheel_radius" value="0.07162" />
+  <xacro:property name="wheel_width" value="0.05" />
   <xacro:property name="wheel_pos_x" value="0.120" />
   <xacro:property name="wheel_pos_y" value="0.1355" />

Commit message: revert back to the original from main branch

File: linorobot2_description/urdf/2wd_properties.urdf.xacro (robot description, xacro)
@@ -21,5 +21,5 @@
   <!-- <xacro:property name="wheel_mesh_file" value="file://$(find linorobot2_description)/meshes/tire.dae" /> -->
   <xacro:property name="laser_pose">
-    <origin xyz="0.0 0 0.17" rpy="0 0 0"/>
+    <origin xyz="0.12 0 0.33" rpy="0 0 0"/>
   </xacro:property>
   <xacro:property name="depth_sensor_pose">

File: linorobot2_description/urdf/controllers/diff_drive.urdf.xacro (robot description, xacro)
@@ -5,5 +5,5 @@
         filename="gz-sim-diff-drive-system"
         name="gz::sim::systems::DiffDrive">
-        <topic>/cmd_vel</topic>
+        <topic>cmd_vel</topic>
         <!-- <frame_id>odom</frame_id> -->
         <child_frame_id>base_footprint</child_frame_id>

File: linorobot2_description/urdf/controllers/omni_drive.urdf.xacro (robot description, xacro)
@@ -5,5 +5,5 @@
         filename="gz-sim-mecanum-drive-system"
         name="gz::sim::systems::MecanumDrive">
-        <topic>/cmd_vel</topic>
+        <topic>cmd_vel</topic>
         <!-- <frame_id>odom</frame_id> -->
         <child_frame_id>base_footprint</child_frame_id>

File: linorobot2_description/urdf/controllers/skid_steer.urdf.xacro (robot description, xacro)
@@ -5,5 +5,5 @@
         filename="gz-sim-diff-drive-system"
         name="gz::sim::systems::DiffDrive">
-          <topic>/cmd_vel</topic>
+          <topic>cmd_vel</topic>
           <!-- <frame_id>odom</frame_id> -->
           <child_frame_id>base_footprint</child_frame_id>
