Commit message: adjusted robomow_612p driving wheels width

File: linorobot2_description/urdf/robomow_612p_properties.urdf.xacro (robot description, xacro)
@@ -7,5 +7,5 @@
   <!-- Driving wheel diameter: 8.5 inch -> radius: 4.25 inch = 0.10795 m -->
   <xacro:property name="wheel_radius" value="0.10795" />
-  <xacro:property name="wheel_width" value="0.05" /> <!-- Estimated value -->
+  <xacro:property name="wheel_width" value="0.090" />
   <!-- Caster wheel position: 19 inch from driving axle = 0.4826 m -->
   <xacro:property name="wheel_pos_x" value="0.0" />
@@ -17,6 +17,6 @@
   <xacro:property name="caster_pos_y" value="0.0" />
   <xacro:property name="caster_pos_z" value="0.0" />
-  <!-- Base dimensions (Estimated based on wheelbase) -->
-  <xacro:property name="base_length" value="0.6" />
+  <!-- Base dimensions -->
+  <xacro:property name="base_length" value="0.71" />
   <xacro:property name="base_height" value="0.15" />
   <xacro:property name="base_mass" value="20.0" />

Commit message: adjust robomow_612p urdf model

File: linorobot2_description/urdf/robomow_612p_properties.urdf.xacro (robot description, xacro)
@@ -11,13 +11,13 @@
   <xacro:property name="wheel_pos_x" value="0.0" />
   <xacro:property name="wheel_pos_y" value="0.2794" /> <!-- base_width / 2 -->
-  <xacro:property name="wheel_pos_z" value="0.0" />
+  <xacro:property name="wheel_pos_z" value="-0.0508" />
   <!-- Caster wheel diameter: 3.5 inch -> radius: 1.75 inch = 0.04445 m -->
   <xacro:property name="caster_radius" value="0.04445" />
-  <xacro:property name="caster_pos_x" value="0.4826" />
+  <xacro:property name="caster_pos_x" value="0.5334" />
   <xacro:property name="caster_pos_y" value="0.0" />
   <xacro:property name="caster_pos_z" value="0.0" />
   <!-- Base dimensions -->
-  <xacro:property name="base_length" value="0.71" />
-  <xacro:property name="base_height" value="0.15" />
+  <xacro:property name="base_length" value="0.737" />
+  <xacro:property name="base_height" value="0.2667" />
   <xacro:property name="base_mass" value="20.0" />
   <xacro:property name="base_mesh_file" value="" />

File: linorobot2_description/urdf/robots/robomow_612p.urdf.xacro (robot description, xacro)
@@ -44,5 +44,5 @@
       side="front"
       mass="0.1"
-      base_length="${base_length}"
+      base_length="${caster_pos_x}"
       wheel_radius="${wheel_radius}"
       wheel_pos_z="${wheel_pos_z}"
