Commit message: working base controllers

File: linorobot2_description/urdf/controllers/omni_drive.urdf.xacro (robot description, xacro)
@@ -1,17 +1,19 @@
 <robot xmlns:xacro="http://ros.org/wiki/xacro">
-  <xacro:macro name="omni_drive_controller">
+  <xacro:macro name="omni_drive_controller" params="wheel_separation wheel_base wheel_radius">
     <gazebo>
-    <plugin name="object_controller" filename="libgazebo_ros_planar_move.so">
-      <ros>
-        <argument>odom:=odom/unfiltered</argument>
-      </ros>
-      <command_topic>cmd_vel</command_topic>
-      <odometry_topic>odom/unfiltered</odometry_topic>
-      <odometry_frame>odom</odometry_frame>
-      <odometry_rate>20.0</odometry_rate>
-      <robot_base_frame>base_footprint</robot_base_frame>
-      <publish_odom>true</publish_odom>
-      <publish_odom_tf>false</publish_odom_tf>
-    </plugin>
+      <plugin
+        filename="ignition-gazebo-mecanum-drive-systems"
+        name="ignition::gazebo::systems::MecanumDrive">
+        <topic>/cmd_vel</topic>
+        <frame_id>odom</frame_id>
+        <child_frame_id>base_footprint</child_frame_id>
+        <odom_topic>odom/unfiltered</odom_topic>
+        <left_joint>left_wheel_joint</left_joint>
+        <right_joint>right_wheel_joint</right_joint>
+        <wheel_separation>${wheel_separation}</wheel_separation>
+        <wheelbase>${wheel_base}</wheelbase>
+        <wheel_radius>${wheel_radius}</wheel_radius>
+        <odom_publish_frequency>50</odom_publish_frequency>
+      </plugin>
   </gazebo>
   </xacro:macro>

File: linorobot2_description/urdf/controllers/skid_steer.urdf.xacro (robot description, xacro)
@@ -1,25 +1,19 @@
 <robot xmlns:xacro="http://ros.org/wiki/xacro">
-  <xacro:macro name="diff_drive_controller" params="wheel_separation wheel_radius wheel_torque">
+  <xacro:macro name="diff_drive_controller" params="wheel_separation wheel_radius">
     <gazebo>
-      <plugin name="differential_drive_controller" filename="libgazebo_ros_diff_drive.so">
-        <ros>
-          <argument>odom:=odom/unfiltered</argument>
-        </ros>
-        <num_wheel_pairs>2</num_wheel_pairs>
+      <plugin
+        filename="ignition-gazebo-diff-drive-system"
+        name="ignition::gazebo::systems::DiffDrive">
+        <topic>/cmd_vel</topic>
+        <frame_id>odom</frame_id>
+        <child_frame_id>base_footprint</child_frame_id>
+        <odom_topic>odom/unfiltered</odom_topic>
+        <left_joint>rear_left_wheel_joint</left_joint>
+        <right_joint>rear_right_wheel_joint</right_joint>
         <left_joint>front_left_wheel_joint</left_joint>
         <right_joint>front_right_wheel_joint</right_joint>
-        <left_joint>rear_left_wheel_joint</left_joint>
-        <right_joint>rear_right_wheel_joint</right_joint>
         <wheel_separation>${wheel_separation}</wheel_separation>
-        <wheel_separation>${wheel_separation}</wheel_separation>
-        <wheel_diameter>${wheel_radius * 2}</wheel_diameter>
-        <wheel_diameter>${wheel_radius * 2}</wheel_diameter>
-        <updateRate>100</updateRate>
-        <max_wheel_acceleration>1.0</max_wheel_acceleration>
-        <robot_base_frame>base_footprint</robot_base_frame>
-        <publish_odom>true</publish_odom>
-        <publish_odom_tf>false</publish_odom_tf>
-        <publish_wheel_tf>true</publish_wheel_tf>
-        <odometry_frame>odom</odometry_frame>
+        <wheel_radius>${wheel_radius}</wheel_radius>
+        <odom_publish_frequency>50</odom_publish_frequency>
       </plugin>
     </gazebo>

File: linorobot2_description/urdf/robots/2wd.urdf.xacro (robot description, xacro)
@@ -5,7 +5,7 @@
   <xacro:include filename="$(find linorobot2_description)/urdf/mech/wheel.urdf.xacro" />
   <xacro:include filename="$(find linorobot2_description)/urdf/mech/caster_wheel.urdf.xacro" />
-  <!-- <xacro:include filename="$(find linorobot2_description)/urdf/sensors/imu.urdf.xacro" />
+  <xacro:include filename="$(find linorobot2_description)/urdf/sensors/imu.urdf.xacro" />
   <xacro:include filename="$(find linorobot2_description)/urdf/sensors/generic_laser.urdf.xacro" />
-  <xacro:include filename="$(find linorobot2_description)/urdf/sensors/depth_sensor.urdf.xacro" /> -->
+  <xacro:include filename="$(find linorobot2_description)/urdf/sensors/depth_sensor.urdf.xacro" />
   <xacro:include filename="$(find linorobot2_description)/urdf/controllers/diff_drive.urdf.xacro" />
   <xacro:base
@@ -53,5 +53,5 @@
     />
   </xacro:if>
-  <!-- <xacro:imu/>
+  <xacro:imu/>
   <xacro:generic_laser>
     <xacro:insert_block name="laser_pose" />
@@ -59,9 +59,8 @@
   <xacro:depth_sensor>
     <xacro:insert_block name="depth_sensor_pose" />
-  </xacro:depth_sensor> -->
+  </xacro:depth_sensor>
   <xacro:diff_drive_controller
     wheel_separation="${wheel_pos_y * 2}"
     wheel_radius="${wheel_radius}"
-    wheel_torque="${wheel_torque}"
   />
 </robot>

File: linorobot2_description/urdf/robots/4wd.urdf.xacro (robot description, xacro)
@@ -62,5 +62,4 @@
     wheel_separation="${wheel_pos_y * 2}"
     wheel_radius="${wheel_radius}"
-    wheel_torque="${wheel_torque}"
   />
 </robot>

File: linorobot2_description/urdf/robots/mecanum.urdf.xacro (robot description, xacro)
@@ -59,4 +59,8 @@
     <xacro:insert_block name="depth_sensor_pose" />
   </xacro:depth_sensor>
-  <xacro:omni_drive_controller/>
+  <xacro:omni_drive_controller
+    wheel_separation="${wheel_pos_y * 2}"
+    wheel_base="${wheel_pos_x * 2}"
+    wheel_radius="${wheel_radius}"
+  />
 </robot>
