Commit message: fixed mecanum controller

File: linorobot2_description/urdf/controllers/diff_drive.urdf.xacro (robot description, xacro)
@@ -1,4 +1,4 @@
 <robot xmlns:xacro="http://ros.org/wiki/xacro">
-  <xacro:macro name="diff_drive_controller" params="wheel_separation wheel_radius wheel_torque">
+  <xacro:macro name="diff_drive_controller" params="wheel_separation wheel_radius">
     <gazebo>
       <plugin

File: linorobot2_description/urdf/controllers/omni_drive.urdf.xacro (robot description, xacro)
@@ -3,5 +3,5 @@
     <gazebo>
       <plugin
-        filename="ignition-gazebo-mecanum-drive-systems"
+        filename="ignition-gazebo-mecanum-drive-system"
         name="ignition::gazebo::systems::MecanumDrive">
         <topic>/cmd_vel</topic>
@@ -9,6 +9,8 @@
         <child_frame_id>base_footprint</child_frame_id>
         <odom_topic>odom/unfiltered</odom_topic>
-        <left_joint>left_wheel_joint</left_joint>
-        <right_joint>right_wheel_joint</right_joint>
+        <front_left_joint>front_left_wheel_joint</front_left_joint>
+        <front_right_joint>front_right_wheel_joint</front_right_joint>
+        <back_left_joint>rear_left_wheel_joint</back_left_joint>
+        <back_right_joint>rear_right_wheel_joint</back_right_joint>
         <wheel_separation>${wheel_separation}</wheel_separation>
         <wheelbase>${wheel_base}</wheelbase>

File: linorobot2_description/urdf/controllers/skid_steer.urdf.xacro (robot description, xacro)
@@ -9,8 +9,8 @@
         <child_frame_id>base_footprint</child_frame_id>
         <odom_topic>odom/unfiltered</odom_topic>
+        <left_joint>front_left_wheel_joint</left_joint>
+        <right_joint>front_right_wheel_joint</right_joint>
         <left_joint>rear_left_wheel_joint</left_joint>
         <right_joint>rear_right_wheel_joint</right_joint>
-        <left_joint>front_left_wheel_joint</left_joint>
-        <right_joint>front_right_wheel_joint</right_joint>
         <wheel_separation>${wheel_separation}</wheel_separation>
         <wheel_radius>${wheel_radius}</wheel_radius>

File: linorobot2_description/urdf/robots/2wd.urdf.xacro (robot description, xacro)
@@ -53,11 +53,11 @@
     />
   </xacro:if>
-  <xacro:imu/>
+  <!-- <xacro:imu/> -->
   <xacro:generic_laser>
     <xacro:insert_block name="laser_pose" />
   </xacro:generic_laser>
-  <xacro:depth_sensor>
+  <!-- <xacro:depth_sensor>
     <xacro:insert_block name="depth_sensor_pose" />
-  </xacro:depth_sensor>
+  </xacro:depth_sensor> -->
   <xacro:diff_drive_controller
     wheel_separation="${wheel_pos_y * 2}"

File: linorobot2_description/urdf/sensors/laser.urdf.xacro (robot description, xacro)
@@ -41,38 +41,32 @@
       <xacro:insert_block name="origin" />
     </joint>
-    <gazebo reference="${frame_id}">
-      <sensor type="ray" name="${frame_id}_head_hokuyo_sensor">
-        <always_on>true</always_on>
-        <update_rate>${update_rate}</update_rate>
-        <pose>0 0 0 0 0 0</pose>
-        <visualize>false</visualize>
-        <ray>
-          <scan>
-            <horizontal>
-              <samples>${ray_count}</samples>
-              <resolution>1</resolution>
-              <min_angle>${min_angle}</min_angle>
-              <max_angle>${max_angle}</max_angle>
-            </horizontal>
-          </scan>
-          <range>
-            <min>${min_range}</min>
-            <max>${max_range}</max>
-            <resolution>0.01</resolution>
-          </range>
-        </ray>
-        <plugin name="${frame_id}_gazebo_ros_head_hokuyo_controller" filename="libgazebo_ros_ray_sensor.so">
-          <ros>
-            <remapping>~/out:=${topic_name}</remapping>
-          </ros>
-          <output_type>sensor_msgs/LaserScan</output_type>
-          <alwaysOn>true</alwaysOn>
-          <updateRate>${update_rate}</updateRate>
-          <topicName>${topic_name}</topicName>
-          <frame_name>${frame_id}</frame_name>
-          <output_type>sensor_msgs/LaserScan</output_type>
-        </plugin>
-      </sensor>
-    </gazebo>
+    <sensor name='gpu_lidar' type='gpu_lidar'>
+      <pose>0 0 0 0 0 0</pose>
+      <topic>scan</topic>
+      <ignition_frame_id>linorbot2/${frame_id}</ignition_frame_id>
+      <update_rate>${update_rate}</update_rate>
+      <lidar>
+        <scan>
+          <horizontal>
+            <samples>${ray_count}</samples>
+            <resolution>1</resolution>
+            <min_angle>${min_angle}</min_angle>
+            <max_angle>${max_angle}</max_angle>
+          </horizontal>
+          <vertical>
+            <samples>1</samples>
+            <resolution>1</resolution>
+            <min_angle>0.0</min_angle>
+            <max_angle>0.0</max_angle>
+          </vertical>
+        </scan>
+        <range>
+          <min>${min_range}</min>
+          <max>${max_range}</max>
+          <resolution>0.01</resolution>
+        </range>
+      </lidar>
+      <visualize>true</visualize>
+    </sensor>
   </xacro:macro>
 </robot>
